File: Souffle_v3_sweep_choc/PCB/Souffle_v3_sweep_choc.kicad_pcb (KiCad board)
At the start: 2 copper layers, 137.2 x 114.5 mm, 84 parts, among them J1 LED, J2 4PIN, J3 OLED, J4 Conn_01x01_Female, J5 Conn_01x01_Female, SW1 SW_PUSH, SW10 SW_PUSH, SW11 SW_PUSH, SW12 SW_PUSH, SW13 SW_PUSH, SW14 SW_PUSH, SW15 SW_PUSH, SW16 SW_PUSH, SW17 SW_PUSH, SW18 SW_PUSH, SW19 SW_PUSH, SW2 SW_PUSH, SW20 SW_PUSH, SW21 SW_PUSH, SW22 SW_PUSH, SW23 SW_PUSH, SW24 SW_PUSH, SW25 SW_PUSH, SW25b1 RotaryEncoder_Switch, SW26 SW_PUSH, SW27 SW_PUSH, SW28 SW_PUSH, SW29 SW_PUSH, SW3 SW_PUSH, SW30 SW_PUSH, SW31 SW_SPDT, SW4 SW_PUSH, SW5 SW_PUSH, SW6 SW_PUSH, SW7 SW_PUSH, SW8 SW_PUSH, SW9 SW_PUSH, U1 ProMicro

Commit message: Updated choc Soufflé.
Parts:
- SW26: footprint SofleKeyboard-footprint:CherryMX_Hotswap_1.5_mod -> SofleKeyboard-footprint:Choc_Hotswap_Souffle
- moved SW6 8.09 mm to (196.1, 64.1)
- moved SW5 7.45 mm to (178.1, 62.6)
- moved SW4 6.91 mm to (160.1, 50.6)
- moved SW12 6.66 mm to (196.1, 81.1)
- moved SW3 6.50 mm to (142.1, 44.4)
- moved SW2 6.24 mm to (124.1, 48.9)
- moved SW1 6.15 mm to (106.1, 51.6)
- moved SW11 5.87 mm to (178.1, 79.6)
- moved SW18 5.64 mm to (196.1, 98.1)
- moved SW30 5.63 mm to (196.1, 132.1)
- moved SW24 5.25 mm to (196.1, 115.1)
- moved SW10 5.17 mm to (160.1, 67.6)
- moved SW17 4.67 mm to (178.1, 96.6)
- moved SW9 4.61 mm to (142.1, 61.4)
- moved SW8 4.23 mm to (124.1, 65.9)
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
Commit message: Checkpoint commit.
Parts:
- moved J1 11.7 mm to (94.0, 78.7), turned to 0 degrees
- moved TH1 9.77 mm to (76.5, 79.2)
- moved J4 3.90 mm to (89.8, 42.6)
- moved J5 3.90 mm to (80.3, 42.6)
- moved U1 3.90 mm to (85.8, 60.1)
- moved J3 3.90 mm to (81.5, 78.7)
- moved JP1 3.90 mm to (89.2, 76.5)
- moved JP2 3.90 mm to (86.6, 76.5)
- moved JP3 3.90 mm to (84.1, 76.5)
- moved JP4 3.90 mm to (81.5, 76.5)
- moved JP5 3.90 mm to (89.2, 76.5)
- moved JP6 3.90 mm to (86.6, 76.5)
- moved JP7 3.90 mm to (84.1, 76.5)
- moved JP8 3.90 mm to (81.5, 76.5)
- moved RSW1 3.84 mm to (88.6, 85.7)
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Routing:
- net row4: track 73.7 -> 18.3 mm
- net BAT: track 96.7 -> 44.3 mm
- net RAW: track 105.7 -> 55.4 mm, vias 3 -> 2
- net ENCB: track 73.3 -> 30.2 mm
- net ENCA: track 75.6 -> 33.2 mm
- net DATA: track 59.0 -> 21.0 mm
- net SW25A: track 54.2 -> 16.8 mm, vias 1 -> 0
- net row3: track 40.0 -> 18.6 mm
- net VCC: track 65.5 -> 50.5 mm
- net LED: track 65.8 -> 52.8 mm
- net SW25B: track 12.3 -> 0.00 mm, vias 1 -> 0
- net col4: track 21.0 -> 15.1 mm, vias 1 -> 0
- net RESET: track 46.1 -> 42.8 mm
- net GND: vias 1 -> 0

Commit message: Checkpoint commit.
Parts:
- TH3, TH4, TH5, TH6, TH7: footprint SofleKeyboard-footprint:HOLE_M2_TH -> SofleKeyboard-footprint:HOLE_M2_TH_CALIBRATED
- moved D12 22.9 mm to (189.9, 89.8)
- moved D11 22.1 mm to (171.4, 87.7)
- moved D10 21.7 mm to (154.6, 76.1)
- moved D9 21.4 mm to (135.6, 69.8)
- moved D8 21.4 mm to (117.8, 74.6)
- moved D7 21.1 mm to (99.5, 77.2)
- moved D24 18.9 mm to (189.6, 123.4)
- moved D23 18.6 mm to (171.3, 121.8)
- moved D21 17.7 mm to (135.7, 104.0)
- moved D20 17.0 mm to (118.0, 108.2)
- moved D22 17.0 mm to (154.5, 109.2)
- moved D19 16.7 mm to (100.0, 110.8)
- moved D30 13.7 mm to (187.7, 135.5), turned to -90 degrees
- moved D5 10.7 mm to (171.8, 70.9)
- moved D3 9.45 mm to (135.6, 53.0)
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
Commit message: Initial routing.
Parts:
- moved D3 20.8 mm to (147.7, 36.1), turned to 180 degrees
- moved D12 20.8 mm to (201.6, 72.7), turned to 180 degrees
- moved D21 20.6 mm to (147.6, 87.2), turned to 180 degrees
- moved D9 20.6 mm to (147.7, 53.2), turned to 180 degrees
- moved D24 20.6 mm to (201.6, 106.7), turned to 180 degrees
- moved D15 20.4 mm to (147.7, 70.1), turned to 180 degrees
- moved D10 20.2 mm to (165.8, 59.3), turned to 180 degrees
- moved D16 20.1 mm to (165.6, 76.2), turned to 180 degrees
- moved D4 20.0 mm to (165.7, 42.3), turned to 180 degrees
- moved D22 19.4 mm to (165.4, 93.2), turned to 180 degrees
- moved D30 18.3 mm to (201.6, 123.7), turned to 180 degrees
- moved D18 16.9 mm to (201.6, 89.7), turned to 180 degrees
- moved D6 16.8 mm to (201.6, 55.7), turned to 180 degrees
- moved D7 16.8 mm to (114.4, 69.6), turned to 90 degrees
- moved D13 16.5 mm to (114.4, 86.5), turned to 90 degrees
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Routing:
- net row3: track 18.6 -> 146.5 mm
- net row1: track 17.9 -> 145.5 mm
- net row0: track 17.9 -> 145.2 mm
- net row2: track 17.9 -> 145.1 mm
- net SW25A: track 16.8 -> 91.9 mm, vias 0 -> 4
- net col0: track 15.1 -> 83.1 mm
- net col1: track 15.2 -> 66.2 mm
- net col3: track 15.5 -> 66.5 mm
- net col2: track 15.1 -> 66.1 mm
- net col4: track 15.1 -> 66.1 mm
- net Net-(D23-Pad2): track 0.00 -> 15.4 mm
- net Net-(D11-Pad2): track 0.00 -> 15.4 mm
- net Net-(D17-Pad2): track 0.00 -> 14.9 mm
- net Net-(D5-Pad2): track 0.00 -> 14.9 mm
- net Net-(D19-Pad2): track 0.00 -> 13.1 mm
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